Commit message: SAVEPOINT

File: CartographerFiles/urdf/StructurePicoDownKit.urdf (robot description, URDF)
Before this commit: robot Structure, 12 links, 11 joints
Links:
- removed link Scan_1_link
- added link laser
Joints:
- joint scanner1_link_joint: child Scan_1_link -> laser; origin xyz=0. 0. 0. rpy=0. 0. 0. -> xyz=0. 0. 0. rpy=0. 0. 1.72

Commit message: added sensor mr18 (choose SensorMode #10 in launch file)

File: CartographerFiles/urdf/StructurePicoDownKit.urdf (robot description, URDF)
Before this commit: robot Structure, 12 links, 11 joints
Links:
- removed link Scan_2_link
- added link mr18_frame
Joints:
- joint scanner2_link_joint: child Scan_2_link -> mr18_frame; origin xyz=0. 0. 0. rpy=0. 0. 2.0943951 -> xyz=0. 0. 0. rpy=3.14159 3.14159 1.72

Commit message: switch urdf to gutte 2

File: CartographerFiles/urdf/StructurePicoDownKit.urdf (robot description, URDF)
Before this commit: robot Structure, 12 links, 11 joints
Joints:
- joint scanner1_link_joint: origin xyz=0. 0. 0. rpy=0. 0. 1.72 -> xyz=0. 0. 0. rpy=0. 0. 3.14
- joint scanner2_link_joint: origin xyz=0. 0. 0. rpy=3.14159 3.14159 1.72 -> xyz=0. 0. 0. rpy=0. 0. 0.
